Commit message: Rename 'root' link to 'base_link' in URDF

File: gg.urdf (robot description, URDF)
Before this commit: robot gg, 424 links, 423 joints
Links:
- removed link root
- added link base_link; visual mesh filename=package://gg/meshes/13480.stl scale=1 1 1; visual mesh filename=package://gg/meshes/13484.stl scale=1 1 1
Joints:
- joint hanging_node_to_root_joint_0: parent root -> base_link
- joint hanging_node_to_root_joint_1: parent root -> base_link
- joint hanging_node_to_root_joint_2: parent root -> base_link
