Commit message: Update robot.urdf

File: description/robot.urdf (robot description, URDF)
Before this commit: robot rossy, 4 links, 3 joints
Links:
- link base_link_chassis: geometry collision box size=0.170 0.190 0.106; collision cylinder length=0.024 radius=0.014
Joints:
- joint base_link_to_base_link_chassis: origin xyz=0 0 0 rpy=0 -0 1.5707 -> xyz=0 0 0 rpy=0 -0 0
- joint left_wheel: origin xyz=0.086 0.0602058 0.0085 rpy=3.14159 -1.5708 0 -> xyz=-0.0602058 0.086 0.0085 rpy=-1.5708 -1.5708 0
- joint right_wheel: origin xyz=-0.086 0.0602058 0.0085 rpy=3.14159 -1.5708 0 -> xyz=-0.0602058 -0.086 0.0085 rpy=-1.5708 -1.5708 0
