Commit message: Update lidar.xacro

File: description/lidar.xacro (robot description, xacro)
@@ -10,5 +10,5 @@
             <origin xyz="0 0 0" rpy="1.5708 -0 -3.14159"/>
             <geometry>
-                <mesh filename="file://$(find rossy)/description/assets/lidar.stl"/>
+                <mesh filename="package://rossy/description/assets/lidar.stl"/>
             </geometry>
             <material name="lidar_material">

Commit message: Update lidar.xacro

File: description/lidar.xacro (robot description, xacro)
@@ -2,5 +2,5 @@
 <robot xmlns:xacro="http://www.ros.org/wiki/xacro" >
     <joint name="laser_joint" type="fixed">
-        <parent link="base_link_chassis"/>
+        <parent link="chassis"/>
         <child link="laser_frame"/>
         <origin xyz="-0.0307058 -0.00250012 0.1371" rpy="0 0 0"/>
@@ -10,5 +10,5 @@
             <origin xyz="0 0 0" rpy="1.5708 -0 -3.14159"/>
             <geometry>
-                <mesh filename="package://rossy/description/assets/lidar.stl"/>
+                <mesh filename="file://$(find rossy)/description/assets/lidar.stl"/>
             </geometry>
             <material name="lidar_material">
@@ -17,4 +17,11 @@
         </visual>
     </link>
+    <gazebo>
+        <plugin
+            filename="gz-sim-sensors-system"
+            name="gz::sim::systems::Sensors">
+            <render_engine>ogre2</render_engine>
+        </plugin>
+    </gazebo>
     <gazebo reference="laser_frame">
         <sensor name="laser" type="gpu_lidar">
@@ -23,5 +30,5 @@
             <visualize>true</visualize>
             <always_on>true</always_on>
-            <update_rate>10</update_rate>
+            <update_rate>20</update_rate>
             <topic>scan</topic>
             <ray>
@@ -34,13 +41,8 @@
                 </scan>
                 <range>
-                    <min>0.3</min>
+                    <min>0.15</min>
                     <max>12</max>
                 </range>
             </ray>
-            <plugin
-                filename="gz-sim-sensors-system"
-                name="gz::sim::systems::Sensors">
-                <render_engine>ogre2</render_engine>
-            </plugin>
         </sensor>
     </gazebo>

Commit message: Update lidar.xacro

File: description/lidar.xacro (robot description, xacro)
@@ -4,16 +4,7 @@
         <parent link="chassis"/>
         <child link="laser_frame"/>
-        <origin xyz="-0.0307058 -0.00250012 0.1371" rpy="0 0 0"/>
+        <origin xyz="-0.0307058 -0.00250012 0.1371" rpy="0 0 3.14159"/>
     </joint>
     <link name="laser_frame">
-        <visual>
-            <origin xyz="0 0 0" rpy="1.5708 -0 -3.14159"/>
-            <geometry>
-                <mesh filename="file://$(find rossy)/description/assets/lidar.stl"/>
-            </geometry>
-            <material name="lidar_material">
-                <color rgba="0.109804 0.109804 0.109804 1"/>
-            </material>
-        </visual>
     </link>
     <gazebo>
