Commit message: Update mesh file paths to use package URI format

File: description/robot_core.urdf (robot description, URDF)
Before this commit: robot description, 4 links, 3 joints
Links:
- link base_link_chassis: geometry collision box size=0.170 0.190 0.106; collision cylinder length=0.024 radius=0.014
- link wheel: geometry collision cylinder length=0.025 radius=0.03; visual mesh filename=package://rossy/description/assets/hex_nut.stl
- link wheel_2: geometry collision cylinder length=0.025 radius=0.03; visual mesh filename=package://rossy/description/assets/hex_nut.stl

Commit message: Update URDF for robot model with new links and joints

File: description/robot_core.urdf (robot description, URDF)
Before this commit: robot description, 4 links, 3 joints
Links:
- removed link base_link_chassis
- added link base_footprint
- added link caster_wheel; collision cylinder length=0.02550 radius=0.014; visual mesh filename=file://$(find rossy)/description/assets/caster_wheel.stl
- added link chassis, mass 0.859503; collision box size=0.170 0.190 0.106; collision cylinder length=0.055 radius=0.045
- link base_link: mass 1e-09 -> 0.1
- link wheel: geometry collision sphere radius=0.034; visual mesh filename=file://$(find rossy)/description/assets/hex_nut.stl
- link wheel_2: geometry collision sphere radius=0.034; visual mesh filename=file://$(find rossy)/description/assets/hex_nut.stl
Joints:
- removed joint base_link_to_base_link_chassis
- added joint base_footprint_joint: type fixed, parent base_link, child base_footprint, origin xyz=0 0 0 rpy=0 0 0
- added joint base_link_to_chassis: type fixed, parent base_link, child chassis, origin xyz=0 0 0 rpy=0 -0 0
- added joint caster_wheel_joint: type fixed, parent chassis, child caster_wheel, origin xyz=0.0397942 0 0 rpy=0.0 0.0 0.0
- joint left_wheel: limit effort=10 velocity=10 -> effort=0.05 velocity=10; parent base_link_chassis -> chassis
- joint right_wheel: limit effort=10 velocity=10 -> effort=0.05 velocity=10; parent base_link_chassis -> chassis

Commit message: Uncomment lidar visual element in URDF

File: description/robot_core.urdf (robot description, URDF)
Before this commit: robot description, 6 links, 5 joints
Links:
- link chassis: geometry collision box size=0.170 0.190 0.106; collision cylinder length=0.055 radius=0.045
